File: 68k-SBC/68kBoardSupervisorShield/68kBoardSupervisorShield.kicad_pcb (KiCad board)
At the start: 2 copper layers, 4 parts, among them J1 ADBUS, J2 SIGBUS

Commit message: Finalized 68kBoard and 68kBoardSupervisorShield
Connections:
- XA1 pad D10: Net-(XA1-PadD10) -> RESET
- XA1 pad D11: Net-(XA1-PadD11) -> BERR
- XA1 pad D30: /A16 -> 0SEL
- XA1 pad D6: RESET -> Net-(XA1-PadD6)
- XA1 pad GND2: Net-(XA1-PadGND2) -> GND
- XA1 pad GND3: Net-(XA1-PadGND3) -> GND
- XA1 pad GND5: Net-(XA1-PadGND5) -> GND
- XA1 pad GND6: Net-(XA1-PadGND6) -> GND
Routing:
- net /A16: track 43.0 -> 0.00 mm
- net 0SEL: track 0.00 -> 32.3 mm
- net BERR: track 0.00 -> 28.0 mm
- net RESET: track 11.9 -> 21.8 mm
- net /D3: track 75.4 -> 76.0 mm
- net BG: track 70.6 -> 71.2 mm
- net /D6: track 64.9 -> 65.5 mm
- net /D4: track 69.5 -> 70.1 mm
- net /D7: track 67.6 -> 68.2 mm
- net /D5: track 71.5 -> 72.1 mm
- net /D2: track 73.4 -> 74.0 mm
- net /D1: track 79.4 -> 80.0 mm
- net /D0: track 78.0 -> 78.6 mm
- net DTACK: track 79.3 -> 79.9 mm
- added copper zone on B.Cu, net GND
- added copper zone on F.Cu, net GND
Other:
- board outline added: 89.9 x 53.3 mm
