File: hardware/68k-SBC/68kBoard/68kBoard.sch (KiCad schematic (older format))
At the start: 38 parts, among them J1 ADBUS, J2 SIGBUS, J3 Barrel_Jack, SW1 RESET, U1 74HC14, U12 74LS32, U2 68000D, U3 L7805, U4 74LS32, U5 74LS393, Y1 Crystal

Commit message: Revision 2 of 68k-SBC
Parts:
- removed U12: 74LS32, Package_DIP:DIP-14_W7.62mm_LongPads, symbol 74xx:74LS32
- removed U5: 74LS393, Package_DIP:DIP-14_W7.62mm_LongPads, symbol 74xx:74LS393
- added C15: 0.47uF, Capacitor_THT:C_Disc_D3.0mm_W2.0mm_P2.50mm, symbol Device:C_Small
- added C9: 0.1uF, Capacitor_THT:C_Disc_D3.0mm_W2.0mm_P2.50mm, symbol Device:C_Small
- added H1, H2, H3, H4: ., MountingHole:MountingHole_2.7mm_Pad_Via, symbol Mechanical:MountingHole
- added HS1: Heatsink, Heatsink:Heatsink_Fischer_SK104-STC-STIC_35x13mm_2xDrill2.5mm, symbol Mechanical:Heatsink
- added R12: 10k, Resistor_THT:R_Axial_DIN0207_L6.3mm_D2.5mm_P7.62mm_Horizontal, symbol Device:R_Small
- added unit 6 of U3
- added U4: 74LS05, Package_DIP:DIP-14_W7.62mm_LongPads, symbol 74xx:74LS05
- added U6: 74LS20, Package_DIP:DIP-14_W7.62mm_LongPads, symbol 74xx:74LS20
- C1: renamed from C3; value 47uF -> 470uF; footprint Capacitor_THT:CP_Radial_D12.5mm_P5.00mm -> Capacitor_THT:CP_Radial_D10.0mm_P5.00mm
- C2: renamed from C10; value 47uF -> 470uF; footprint Capacitor_THT:CP_Radial_D12.5mm_P5.00mm -> Capacitor_THT:CP_Radial_D10.0mm_P5.00mm
- U1: renamed from U3; footprint Package_TO_SOT_THT:TO-220-3_Horizontal_TabDown -> Package_TO_SOT_THT:TO-220-3_Vertical
- U2: value 68000D -> 68010
- renumbered C2 to C10, C5 to C11, C7 to C12, C9 to C13, C12 to C14, C13 to C3, C1 to C4, C4 to C5, C8 to C7, C11 to C8, J3 to J2, J2 to J3, R13 to R10, R7 to R11, R2 to R13, R8 to R14, R3 to R2, R4 to R3, R5 to R4, R9 to R5, R10 to R6, R6 to R7, R11 to R8, R12 to R9, U1 to U3, U4 to U5
Connections:
- net labels added: IACK, IP4, IP5
- net labels removed: IP2, IP3, SIACK, SIRQ
- wire segments 240 -> 258
- no-connect marks 4 -> 5
Other:
- moved on the sheet: C1, C10, C11, C12, C13, C14, C2, C3, C4, C5, C6, C7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
