File: hardware/68k-SBC/68kBoard/Memory.sch (KiCad schematic (older format))
At the start: 13 parts, among them Q1 Q_NMOS_SGD, U1 74HC14, U10 HM628512, U12 74LS32, U13 74LS32, U4 74LS32, U5 74LS393, U6 74LS138, U7 28C256, U8 28C256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

Commit message: Updated readme
Parts:
- removed U7, U8: 28C256, Package_DIP:DIP-28_W15.24mm_Socket_LongPads, symbol Memory_EEPROM:28C256
- added JP?: ROMACK, Connector_PinHeader_2.54mm:PinHeader_1x03_P2.54mm_Vertical, symbol Jumper:Jumper_3_Bridged12
- added Q?: Q_NMOS_SGD, Package_TO_SOT_THT:TO-92, symbol Device:Q_NMOS_SGD
- added unit 4 of U12
- added U? (x2): AM29F040, symbol ComputieParts:AM29F040
- added U? (x3): 74HC14, Package_DIP:DIP-14_W7.62mm_LongPads, symbol 74xx:74HC14
- added U?: 74LS20, symbol 74xx:74LS20
- renumbered U13 to U12
Connections:
- net labels added: ROMSEL-L, ROMSEL-U
- wire segments 158 -> 194
Other:
- moved on the sheet: U12A, U12B, U9

Commit message: Revision 2 of 68k-SBC
Parts:
- removed JP1: ROMACK, Connector_PinHeader_2.54mm:PinHeader_1x03_P2.54mm_Vertical, symbol Jumper:Jumper_3_Bridged12
- removed Q1, Q?: Q_NMOS_SGD, Package_TO_SOT_THT:TO-92, symbol Device:Q_NMOS_SGD
- removed U1, U?: 74HC14, Package_DIP:DIP-14_W7.62mm_LongPads, symbol 74xx:74HC14
- removed U4: 74LS32, Package_DIP:DIP-14_W7.62mm_LongPads, symbol 74xx:74LS32
- removed U5: 74LS393, Package_DIP:DIP-14_W7.62mm_LongPads, symbol 74xx:74LS393
- added R15: 10k, Resistor_THT:R_Axial_DIN0207_L6.3mm_D2.5mm_P7.62mm_Horizontal, symbol Device:R_Small
- added U4: 74LS05, Package_DIP:DIP-14_W7.62mm_LongPads, symbol 74xx:74LS05
- U6: renamed from U?; footprint (none) -> Package_DIP:DIP-14_W7.62mm_LongPads
- U8, U9: renamed from U?; footprint (none) -> Package_DIP:DIP-32_W15.24mm_Socket_LongPads
- gave numbers to parts that had none: 2
- renumbered JP2 to JP1, U9 to U10, U10 to U11, U12 to U5, U6 to U7
Connections:
- net labels added: RD-L, RD-U, WR-L, WR-U
- net labels removed: CLK, ROMSEL-L, ROMSEL-U
- wire segments 194 -> 175
- no-connect marks 3 -> 0
Other:
- moved on the sheet: JP1, JP2, U5A, U5D, U6A, U7
