File: hardware/68k-SBC/68kBoard/UART.sch (KiCad schematic (older format))
At the start: 20 parts, among them J4 Serial1, J5 Serial2, SW2 IP4, SW3 IP5, U11 68681, Y2 Crystal

Commit message: Revision 2 of 68k-SBC
Parts:
- added JP5: IRQ, Connector_PinHeader_2.54mm:PinHeader_1x02_P2.54mm_Vertical, symbol Device:Jumper
- added JP6: IACK, Connector_PinHeader_2.54mm:PinHeader_1x02_P2.54mm_Vertical, symbol Device:Jumper
- added TP1: IP2, TestPoint:TestPoint_THTPad_2.0x2.0mm_Drill1.0mm, symbol Connector:TestPoint
- added TP2: IP3, TestPoint:TestPoint_THTPad_2.0x2.0mm_Drill1.0mm, symbol Connector:TestPoint
- added U6: 74LS20, Package_DIP:DIP-14_W7.62mm_LongPads, symbol 74xx:74LS20
- C16: renamed from C14; value 22pF -> 15pF
- C17: renamed from C15; value 22pF -> 5pF
- SW2: value IP4 -> IP2
- SW3: value IP5 -> IP3
- renumbered D4 to D2, D2 to D3, D5 to D4, D3 to D5, R18 to R16, R16 to R17, R19 to R18, R17 to R19, R14 to R20, R15 to R21, U11 to U12
Connections:
- net IP2 is gone; now on an unnamed net: U12.36 (IP2)
- net IP3 is gone; now on an unnamed net: U12.2 (IP3)
- net +5V: now also U6.13
- net SIACK: now also JP6.2
- net SIRQ: now also JP5.1
- net at R20.1, SW3.1: now also TP2.1; no longer U12.38 (IP5)
- net at R21.1, SW2.1: now also TP1.1; no longer U12.39 (IP4)
- new net FC0: U6.9
- new net FC1: U6.10
- new net FC2: U6.12
- new net IACK: JP6.1, U6.8
- new net IP4: U12.39 (IP4)
- new net IP5: U12.38 (IP5)
- new net IPL1: JP5.2
Other:
- moved on the sheet: C16, C17, D2, D3, D4, D5, J4, J5, JP3, JP4, R16, R17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
