File: hardware/68k-SBC/68kBoard/68kBoard.kicad_pcb (KiCad board)
At the start: 2 copper layers, 154.9 x 134.6 mm, 69 parts, among them J1 ADBUS, J2 SIGBUS, J3 Barrel_Jack, J4 Serial1, J5 Serial2, Q1 Q_NMOS_DGS, SW1 RESET, SW2 IP4, SW3 IP5, U1 74HC14, U10 HM628512, U11 68681, U2 68000D, U3 L7805, U4 74LS32, U5 74LS393, U6 74LS138, U7 28C256, U8 28C256, U9 HM628512, Y1 Crystal, Y2 Crystal

Commit message: Updated readme
Other:
- board text added: "68k-SBC Rev. 2"
- board text removed: "68k-SBC Rev. 0"

Commit message: Revision 2 of 68k-SBC
Parts:
- removed ? (x4): , MountingHole:MountingHole_2.7mm_Pad_Via
- removed the C1 at (140.5, 78.7)
- removed the C11 at (168.4, 128.0)
- removed the C2 at (153.2, 128.0)
- removed Q1: Q_NMOS_DGS, Package_TO_SOT_THT:TO-92
- removed the R2 at (120.1, 143.8)
- removed the R8 at (116.3, 136.1)
- added C10: 0.1uF, Capacitor_THT:C_Disc_D3.0mm_W2.0mm_P2.50mm, F.Cu at (155.7, 130.3)
- added C13: 0.1uF, Capacitor_THT:C_Disc_D3.0mm_W2.0mm_P2.50mm, F.Cu at (87.9, 141.5)
- added C14: 0.1uF, Capacitor_THT:C_Disc_D3.0mm_W2.0mm_P2.50mm, F.Cu at (130.3, 130.3)
- added C15: 0.47uF, Capacitor_THT:C_Disc_D3.0mm_W2.0mm_P2.50mm, F.Cu at (96.6, 113.8)
- added C5: 0.1uF, Capacitor_THT:C_Disc_D3.0mm_W2.0mm_P2.50mm, F.Cu at (183.7, 130.3)
- added H1: ., MountingHole:MountingHole_2.7mm_Pad_Via, F.Cu at (60.2, 26.9)
- added H2: ., MountingHole:MountingHole_2.7mm_Pad_Via, F.Cu at (206.5, 26.9)
- added H3: ., MountingHole:MountingHole_2.7mm_Pad_Via, F.Cu at (60.2, 158.0)
- added H4: ., MountingHole:MountingHole_2.7mm_Pad_Via, F.Cu at (206.5, 158.0)
- added HS1: Heatsink, Heatsink:Heatsink_Fischer_SK104-STC-STIC_35x13mm_2xDrill2.5mm, F.Cu at (90.4, 150.6)
- added JP5: IRQ, Connector_PinHeader_2.54mm:PinHeader_1x02_P2.54mm_Vertical, F.Cu at (105.4, 133.4)
- added JP6: IACK, Connector_PinHeader_2.54mm:PinHeader_1x02_P2.54mm_Vertical, F.Cu at (101.8, 133.4)
- added R12: 10k, Resistor_THT:R_Axial_DIN0207_L6.3mm_D2.5mm_P7.62mm_Horizontal, F.Cu at (91.4, 117.3)
- added R13: 5.1k, Resistor_THT:R_Axial_DIN0207_L6.3mm_D2.5mm_P7.62mm_Horizontal, F.Cu at (119.4, 127.3)
- added R14: 5.1k, Resistor_THT:R_Axial_DIN0207_L6.3mm_D2.5mm_P7.62mm_Horizontal, F.Cu at (115.6, 134.9)
- added R15: 10k, Resistor_THT:R_Axial_DIN0207_L6.3mm_D2.5mm_P7.62mm_Horizontal, F.Cu at (130.3, 126.7)
- added TP1: IP2, TestPoint:TestPoint_THTPad_2.0x2.0mm_Drill1.0mm, F.Cu at (58.7, 111.5)
- added TP2: IP3, TestPoint:TestPoint_THTPad_2.0x2.0mm_Drill1.0mm, F.Cu at (58.7, 121.9)
- added U11: HM628512, Package_DIP:DIP-32_W15.24mm_Socket_LongPads, F.Cu at (168.4, 82.8)
- C1: renamed from C3; value 47uF -> 470uF; footprint Capacitor_THT:CP_Radial_D12.5mm_P5.00mm -> Capacitor_THT:CP_Radial_D10.0mm_P5.00mm
- C16: renamed from C14; value 22pF -> 15pF
- C17: renamed from C15; value 22pF -> 5pF
- C2: renamed from C10; value 47uF -> 470uF; footprint Capacitor_THT:CP_Radial_D12.5mm_P5.00mm -> Capacitor_THT:CP_Radial_D10.0mm_P5.00mm
- JP1: value ROMACK -> ROMJMP
- JP2: value ROMJMP -> ROMACK
- SW2: value IP4 -> IP2
- SW3: value IP5 -> IP3
- U1: value 74HC14 -> L7805; footprint Package_DIP:DIP-14_W7.62mm_LongPads -> Package_TO_SOT_THT:TO-220-3_Vertical
- U2: value 68000D -> 68010
- U3: value L7805 -> 74HC14; footprint Package_TO_SOT_THT:TO-220-3_Horizontal_TabDown -> Package_DIP:DIP-14_W7.62mm_LongPads
- U4: value 74LS32 -> 74LS05
- U5: value 74LS393 -> 74LS32
- U6: value 74LS138 -> 74LS20; footprint Package_DIP:DIP-16_W7.62mm_LongPads -> Package_DIP:DIP-14_W7.62mm_LongPads
- U7: value 28C256 -> 74LS138; footprint Package_DIP:DIP-28_W15.24mm_Socket_LongPads -> Package_DIP:DIP-16_W7.62mm_LongPads
- U8: value 28C256 -> AM29F040; footprint Package_DIP:DIP-28_W15.24mm_Socket_LongPads -> Package_DIP:DIP-32_W15.24mm_Socket_LongPads
- U9: value HM628512 -> AM29F040
- moved U7 97.0 mm to (176.0, 133.3)
- moved C4 67.7 mm to (140.5, 75.9)
- moved C8 55.2 mm to (168.4, 130.3)
- moved C12 54.5 mm to (162.8, 79.5)
- moved U9 47.5 mm to (168.4, 37.8)
- moved C9 44.1 mm to (143.0, 130.3), turned to 0 degrees
- moved U1 40.3 mm to (93.0, 146.3), turned to 180 degrees
- moved U3 29.0 mm to (122.7, 133.3), turned to 0 degrees
- moved U4 25.5 mm to (135.4, 133.3)
- moved C2 25.2 mm to (78.5, 138.4)
- moved C1 22.5 mm to (65.3, 138.4)
- moved U8 21.0 mm to (147.6, 37.8)
- moved C7 21.0 mm to (183.6, 79.5)
- moved U10 21.0 mm to (147.6, 82.8)
- moved U6 15.4 mm to (160.8, 133.3)
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- renumbered C5 to C11, C13 to C3, D4 to D2, D2 to D3, D5 to D4, D3 to D5, J3 to J2, J2 to J3, R13 to R10, R7 to R11, R18 to R16, R16 to R17, R19 to R18, R17 to R19, R3 to R2, R14 to R20, R15 to R21, R4 to R3, R5 to R4, R9 to R5, R10 to R6, R6 to R7, R11 to R8, R12 to R9, U11 to U12
Connections:
- C1 pad 1: Net-(C3-Pad1) -> Net-(C1-Pad1)
- J2 pad 1: Net-(C3-Pad1) -> Net-(C1-Pad1)
- J3 pad 28: SIACK -> IACK
- J3 pad 30: SIRQ -> Net-(J3-Pad30)
- J3 pad 36: IP2 -> IP4
- J3 pad 38: IP3 -> IP5
- JP1 pad 2: Net-(JP1-Pad2) -> ROMSEL
- JP1 pad 3: +5V -> 2SEL
- JP2 pad 2: ROMSEL -> Net-(JP2-Pad2)
- JP2 pad 3: 2SEL -> +5V
- R20 pad 1: Net-(R14-Pad1) -> Net-(R20-Pad1)
- R21 pad 1: Net-(R15-Pad1) -> Net-(R21-Pad1)
- SW1 pad 2: RESET -> Net-(C15-Pad1)
- SW2 pad 1: Net-(R15-Pad1) -> Net-(R21-Pad1)
- SW3 pad 1: Net-(R14-Pad1) -> Net-(R20-Pad1)
- U1 pad 1: (no net) -> Net-(C1-Pad1)
- U1 pad 2: (no net) -> GND
- U1 pad 3: Net-(R2-Pad2) -> +5V
- U10 pad 13: D8 -> D0
- U10 pad 14: D9 -> D1
- U10 pad 15: D10 -> D2
- U10 pad 17: D11 -> D3
- U10 pad 18: D12 -> D4
- U10 pad 19: D13 -> D5
- U10 pad 20: D14 -> D6
- U10 pad 21: D15 -> D7
- U10 pad 24: RD -> RD-L
- U10 pad 29: R~W -> WR-L
- U12 pad 2: IP3 -> Net-(R20-Pad1)
- U12 pad 36: IP2 -> Net-(R21-Pad1)
- U12 pad 38: Net-(R14-Pad1) -> IP5
- U12 pad 39: Net-(R15-Pad1) -> IP4
- U3 pad 1: Net-(C3-Pad1) -> R~W
- U3 pad 2: GND -> RD
- U3 pad 3: +5V -> Net-(R13-Pad2)
- U4 pad 1: AS -> Net-(U3-Pad12)
- U4 pad 10: Net-(U1-Pad10) -> DTACK
- U4 pad 11: (no net) -> Net-(R15-Pad2)
- U4 pad 12: (no net) -> Net-(R15-Pad2)
- U4 pad 13: (no net) -> Net-(U4-Pad13)
- U4 pad 2: A23 -> HALT
- U4 pad 3: Net-(U4-Pad3) -> Net-(U3-Pad12)
- U4 pad 4: Net-(U4-Pad3) -> RESET
- U4 pad 5: Net-(U4-Pad5) -> (no net)
- U4 pad 6: Net-(U4-Pad6) -> (no net)
- U4 pad 8: Net-(U4-Pad5) -> (no net)
- U4 pad 9: Net-(U1-Pad8) -> (no net)
- U5 pad 1: CLK -> RD
- U5 pad 10: (no net) -> UDS
- U5 pad 11: (no net) -> WR-U
- U5 pad 12: (no net) -> R~W
- U5 pad 13: (no net) -> UDS
- U5 pad 2: Net-(U4-Pad6) -> LDS
- U5 pad 3: Net-(U5-Pad3) -> RD-L
- U5 pad 4: Net-(Q1-Pad2) -> R~W
- U5 pad 5: Net-(U5-Pad5) -> LDS
- U5 pad 6: Net-(U5-Pad6) -> WR-L
- U5 pad 8: (no net) -> RD-U
- U5 pad 9: (no net) -> RD
- U6 pad 1: A20 -> Net-(U3-Pad10)
- U6 pad 10: 5SEL -> FC1
- U6 pad 11: 4SEL -> (no net)
- U6 pad 12: 3SEL -> FC2
- U6 pad 13: 2SEL -> +5V
- U6 pad 14: RAMSEL -> +5V
- U6 pad 2: A21 -> Net-(U3-Pad8)
- U6 pad 3: A22 -> (no net)
- U6 pad 4: AS -> IOSEL
- U6 pad 5: A23 -> Net-(JP2-Pad2)
- U6 pad 6: +5V -> Net-(U4-Pad13)
- U6 pad 7: IOSEL -> GND
- U6 pad 8: GND -> IACK
- U6 pad 9: 6SEL -> FC0
- U7 pad 1: A15 -> A20
- U7 pad 10: A1 -> 5SEL
- U7 pad 11: D0 -> 4SEL
- U7 pad 12: D1 -> 3SEL
- U7 pad 13: D2 -> 2SEL
- U7 pad 14: GND -> RAMSEL
- U7 pad 15: D3 -> 0SEL
- U7 pad 16: D4 -> +5V
- U7 pad 2: A13 -> A21
- U7 pad 3: A8 -> A22
- U7 pad 4: A7 -> AS
- U7 pad 5: A6 -> A23
- U7 pad 6: A5 -> +5V
- U7 pad 7: A4 -> IOSEL
- U7 pad 8: A3 -> GND
- U7 pad 9: A2 -> 6SEL
- U8 pad 1: A15 -> A19
- U8 pad 10: A1 -> A3
- U8 pad 11: D8 -> A2
- U8 pad 12: D9 -> A1
- U8 pad 13: D10 -> D0
- U8 pad 14: GND -> D1
- U8 pad 15: D11 -> D2
- U8 pad 16: D12 -> GND
- U8 pad 17: D13 -> D3
- U8 pad 18: D14 -> D4
- U8 pad 19: D15 -> D5
- U8 pad 2: A13 -> A17
- U8 pad 20: ROMSEL -> D6
- U8 pad 21: A11 -> D7
- U8 pad 22: RD -> ROMSEL
- U8 pad 23: A12 -> A11
- U8 pad 24: A10 -> RD-L
- U8 pad 25: A9 -> A12
- U8 pad 26: A14 -> A10
- U8 pad 27: R~W -> A9
- U8 pad 28: +5V -> A14
- U8 pad 3: A8 -> A16
- U8 pad 4: A7 -> A13
- U8 pad 5: A6 -> A8
- U8 pad 6: A5 -> A7
- U8 pad 7: A4 -> A6
- U8 pad 8: A3 -> A5
- U8 pad 9: A2 -> A4
- U9 pad 13: D0 -> D8
- U9 pad 14: D1 -> D9
- U9 pad 15: D2 -> D10
- U9 pad 17: D3 -> D11
- U9 pad 18: D4 -> D12
- U9 pad 19: D5 -> D13
- U9 pad 20: D6 -> D14
- U9 pad 21: D7 -> D15
- U9 pad 22: RAMSEL -> ROMSEL
- U9 pad 24: RD -> RD-U
- U9 pad 29: R~W -> A15
- U9 pad 3: A15 -> A16
- U9 pad 31: A16 -> WR-U
- Y1 pad 1: Net-(R2-Pad2) -> Net-(R13-Pad2)
Routing:
- net IP4: track 0.00 -> 238.2 mm, vias 0 -> 1
- net IP5: track 0.00 -> 231.4 mm, vias 0 -> 1
- net IP2: track 222.4 -> 0.00 mm, vias 1 -> 0
- net IP3: track 219.5 -> 0.00 mm, vias 1 -> 0
- net IACK: track 0.00 -> 194.0 mm, vias 0 -> 1
- net SIACK: track 242.6 -> 104.3 mm
- net WR-U: track 0.00 -> 137.5 mm, vias 0 -> 4
- net SIRQ: track 201.9 -> 70.3 mm
- net RD-U: track 0.00 -> 129.3 mm, vias 0 -> 4
- net WR-L: track 0.00 -> 127.8 mm, vias 0 -> 2
- net Net-(R20-Pad1): track 0.00 -> 124.4 mm, vias 0 -> 2
- net UDS: track 186.6 -> 309.8 mm, vias 1 -> 4
- net LDS: track 189.0 -> 300.3 mm, vias 1 -> 4
- net Net-(R14-Pad1): track 106.2 -> 0.00 mm, vias 1 -> 0
- net RD-L: track 0.00 -> 101.6 mm, vias 0 -> 2
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Other:
- board size 154.9 x 134.6 mm -> 154.9 x 139.7 mm
- board text added: "CS"
- board text added: "IACK"
- board text added: "IP0"
- board text added: "IP1"
- board text added: "IP4"
- board text added: "IP5"
- board text added: "IRQ"
- board text added: "OE"
- board text added: "OP0"
- board text added: "OP1"
- board text added: "OP4"
- board text added: "OP5"
- board text added: "OP6"
- board text added: "OP7"
- board text added: "R/W"
- board text added: "RST"
- board text added: "RXA"
- board text added: "RXB"
- board text added: "TXA"
- board text added: "TXB"
- board text added: "WE"
- board text added: "X1"
- board text added: "X2"
- board text removed: "SIACK"
- board text removed: "SIRQ"

Commit message: Final version of rev 2
Parts:
- moved R15 1.02 mm to (130.3, 125.7)
Routing:
- net Net-(R15-Pad2): track 16.3 -> 17.3 mm
- net +5V: track 838.5 -> 839.5 mm
- net AS: track 268.6 -> 269.5 mm
- net A23: track 274.4 -> 275.4 mm
- net GND: track 844.0 -> 844.7 mm
