File: hardware/68k-SBC/68kBoardSupervisorShield/68kBoardSupervisorShield.sch (KiCad schematic (older format))
At the start: 4 parts, among them J1 ADBUS, J2 SIGBUS

Commit message: Revision 2 of 68k-SBC
Parts:
- added J3: UNMAPPED, Connector_PinHeader_2.54mm:PinHeader_2x06_P2.54mm_Vertical, symbol Connector_Generic:Conn_02x06_Odd_Even
- added SW1: RESET, Button_Switch_THT:SW_PUSH_6mm, symbol Switch:SW_Push
Connections:
- net 0SEL: no longer XA1.D30
- net A16: now also XA1.D30
- net A17: now also XA1.A0
- net A18: now also XA1.A1
- net A19: now also XA1.A2
- net A20: now also XA1.A3
- net A21: now also XA1.A4
- net A22: now also XA1.A5
- net A23: now also XA1.A6
- net CLK: now also J3.1 (Pin_1)
- net FC0: now also J3.2 (Pin_2)
- net FC1: now also J3.4 (Pin_4)
- net FC2: now also J3.6 (Pin_6)
- net GND: now also SW1.1
- net HALT: now also XA1.D12
- net IPL0: now also J3.8 (Pin_8)
- net IPL1: now also J3.10 (Pin_10)
- net IPL2: now also J3.12 (Pin_12)
- net OP2: now also J3.9 (Pin_9)
- net OP3: now also J3.7 (Pin_7)
- net ROMSEL: now also XA1.A7
- net at XA1.RST1 (RESET): now also SW1.2
- net IP2 renamed IP4
- net IP4: now also J3.5 (Pin_5)
- net IP3 renamed IP5
- net IP5: now also J3.3 (Pin_3)
- net SIACK renamed IACK
- net IACK: now also J3.11 (Pin_11)
- net SIRQ: no longer names the net of J2.30 (Pin_30)
- no-connect marks 2 -> 5
Other:
- moved on the sheet: J1, J2, JP1
