File: hardware/68k-SBC/68kBoardSupervisorShield/68kBoardSupervisorShield.kicad_pcb (KiCad board)
At the start: 2 copper layers, 89.9 x 53.3 mm, 4 parts, among them J1 ADBUS, J2 SIGBUS

Commit message: Revision 2 of 68k-SBC
Parts:
- added J3: UNMAPPED, Connector_PinHeader_2.54mm:PinHeader_2x06_P2.54mm_Vertical, F.Cu at (108.7, 83.6)
- added SW1: RESET, Button_Switch_THT:SW_PUSH_6mm, F.Cu at (81.3, 101.3)
- moved JP1 4.57 mm to (90.7, 89.4)
Connections:
- net SIRQ renamed Net-(J2-Pad30)
- J2 pad 28: SIACK -> IACK
- J2 pad 36: IP2 -> IP4
- J2 pad 38: IP3 -> IP5
- XA1 pad A0: Net-(XA1-PadA0) -> /A17
- XA1 pad A1: Net-(XA1-PadA1) -> /A18
- XA1 pad A2: Net-(XA1-PadA2) -> /A19
- XA1 pad A3: Net-(XA1-PadA3) -> /A20
- XA1 pad A4: Net-(XA1-PadA4) -> /A21
- XA1 pad A5: Net-(XA1-PadA5) -> /A22
- XA1 pad A6: Net-(XA1-PadA6) -> /A23
- XA1 pad A7: Net-(XA1-PadA7) -> ROMSEL
- XA1 pad D12: Net-(XA1-PadD12) -> HALT
- XA1 pad D30: 0SEL -> /A16
Routing:
- net ROMSEL: track 0.00 -> 111.7 mm
- net /A16: track 0.00 -> 63.3 mm
- net CLK: track 0.00 -> 49.7 mm
- net IP5: track 0.00 -> 48.7 mm
- net GND: track 64.9 -> 107.5 mm
- net IP4: track 0.00 -> 41.6 mm
- net OP3: track 0.00 -> 36.3 mm
- net /A22: track 0.00 -> 32.7 mm, vias 0 -> 1
- net 0SEL: track 32.3 -> 0.00 mm
- net /A17: track 0.00 -> 31.6 mm, vias 0 -> 1
- net OP2: track 0.00 -> 30.7 mm
- net /A19: track 0.00 -> 30.7 mm, vias 0 -> 1
- net /A21: track 0.00 -> 28.3 mm, vias 0 -> 1
- net /A18: track 0.00 -> 28.3 mm, vias 0 -> 1
- net /A20: track 0.00 -> 26.9 mm, vias 0 -> 1
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Other:
- board text added: "+5V"
- board text added: "0SEL"
- board text added: "2SEL"
- board text added: "3SEL"
- board text added: "4SEL"
- board text added: "5SEL"
- board text added: "6SEL"
- board text added: "A1"
- board text added: "A10"
- board text added: "A11"
- board text added: "A12"
- board text added: "A13"
- board text added: "A14"
- board text added: "A15"
- board text added: "A16"
- board text added: "A17"
- board text added: "A18"
- board text added: "A19"
- board text added: "A2"
- board text added: "A20"
- board text added: "A21"
- board text added: "A22"
- board text added: "A23"
- board text added: "A3"
- board text added: "A4"
- board text added: "A5"
- board text added: "A6"
- board text added: "A7"
- board text added: "A8"
- board text added: "A9"
- board text added: "AS"
- board text added: "BERR"
- board text added: "BG"
- board text added: "BGACK"
- board text added: "BR"
- board text added: "CLK"
- board text added: "D0"
- board text added: "D1"
- board text added: "D10"
- board text added: "D11"
- board text added: "D12"
- board text added: "D13"
- board text added: "D14"
- board text added: "D15"
- board text added: "D2"
- board text added: "D3"
- board text added: "D4"
- board text added: "D5"
- board text added: "D6"
- board text added: "D7"
- board text added: "D8"
- board text added: "D9"
- board text added: "DTACK"
- board text added: "FC0"
- board text added: "FC1"
- board text added: "FC2"
- board text added: "GND"
- board text added: "HALT"
- board text added: "IACK"
- board text added: "IOSEL"
- board text added: "IP4"
- board text added: "IP5"
- board text added: "IPL0"
- board text added: "IPL1"
- board text added: "IPL2"
- board text added: "LDS"
- board text added: "OP2"
- board text added: "OP3"
- board text added: "R/~W"
- board text added: "RAMSEL"
- board text added: "RD"
- board text added: "RESET"
- board text added: "ROMSEL"
- board text added: "RST"
- board text added: "UDS"
- board text added: "WR"
