File: hardware/68k-SMT/CompactFlash.sch (KiCad schematic (older format))
At the start: 2 parts, among them J6 CompactFlash, U1 74HC32

Commit message: Removed IDE header which doesn't easily fit, and cleaned up the PCB design a bit
Connections:
- net A11 renamed A4
- net A12 renamed A5
Changed lines of the file:
@@
 	3900 2650 3800 2550
 Text Label 3900 2650 0    50   ~ 0
-A11
+A4
 Wire Wire Line
 	4800 2650 3900 2650
@@
 	6200 2650 6300 2550
 Text Label 6200 2650 2    50   ~ 0
-A12
+A5
 Wire Wire Line
 	6200 2650 5300 2650
