File: hardware/k30-SBC/Logic.sch (KiCad schematic (older format))
At the start: 14 parts, among them SW2 SW_DIP_x06, U10 74LS253, U11 74HC138, U12 74LS393, U2 74HC14, U3 74HC05, U4 74LS139, U5 4072, U6 74HC20, U7 74LS32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

Commit message: Almost completed k30-SBC board design
Parts:
- U10, U9: value 74LS253 -> 74HC253
- U12: value 74LS393 -> 74HC393
- U4: value 74LS139 -> 74HC139
- U7: value 74LS32 -> 74HC32
- U8: value 74LS08 -> 74HC08
Changed lines of the file:
@@
 P 1600 1250
 F 0 "U4" H 1600 1617 50  0000 C CNN
-F 1 "74LS139" H 1600 1526 50  0000 C CNN
+F 1 "74HC139" H 1600 1526 50  0000 C CNN
 F 2 "Package_SO:TSSOP-16_4.4x5mm_P0.65mm" H 1600 1250 50  0001 C CNN
 F 3 "http://www.ti.com/lit/ds/symlink/sn74ls139a.pdf" H 1600 1250 50  0001 C CNN
@@
 P 2800 1350
 F 0 "U8" H 2800 1675 50  0000 C CNN
-F 1 "74LS08" H 2800 1584 50  0000 C CNN
+F 1 "74HC08" H 2800 1584 50  0000 C CNN
 F 2 "Package_SO:TSSOP-14_4.4x5mm_P0.65mm" H 2800 1350 50  0001 C CNN
 F 3 "http://www.ti.com/lit/gpn/sn74LS08" H 2800 1350 50  0001 C CNN
@@
 P 2800 2650
 F 0 "U8" H 2800 2975 50  0000 C CNN
-F 1 "74LS08" H 2800 2884 50  0000 C CNN
+F 1 "74HC08" H 2800 2884 50  0000 C CNN
 F 2 "Package_SO:TSSOP-14_4.4x5mm_P0.65mm" H 2800 2650 50  0001 C CNN
 F 3 "http://www.ti.com/lit/gpn/sn74LS08" H 2800 2650 50  0001 C CNN
@@
 P 2800 2000
 F 0 "U8" H 2800 2325 50  0000 C CNN
-F 1 "74LS08" H 2800 2234 50  0000 C CNN
+F 1 "74HC08" H 2800 2234 50  0000 C CNN
 F 2 "Package_SO:TSSOP-14_4.4x5mm_P0.65mm" H 2800 2000 50  0001 C CNN
 F 3 "http://www.ti.com/lit/gpn/sn74LS08" H 2800 2000 50  0001 C CNN
@@
 P 4500 2000
 F 0 "U9" H 4500 3181 50  0000 C CNN
-F 1 "74LS253" H 4500 3090 50  0000 C CNN
+F 1 "74HC253" H 4500 3090 50  0000 C CNN
 F 2 "Package_SO:SSOP-16_3.9x4.9mm_P0.635mm" H 4500 2000 50  0001 C CNN
 F 3 "http://www.ti.com/lit/gpn/sn74LS253" H 4500 2000 50  0001 C CNN
@@
 P 4500 4650
 F 0 "U10" H 4500 5831 50  0000 C CNN
-F 1 "74LS253" H 4500 5740 50  0000 C CNN
+F 1 "74HC253" H 4500 5740 50  0000 C CNN
 F 2 "Package_SO:SSOP-16_3.9x4.9mm_P0.635mm" H 4500 4650 50  0001 C CNN
 F 3 "http://www.ti.com/lit/gpn/sn74LS253" H 4500 4650 50  0001 C CNN
@@
 AR Path="/613AFF13/6152D712" Ref="U12"  Part="1"
 F 0 "U12" H 7650 2217 50  0000 C CNN
-F 1 "74LS393" H 7650 2126 50  0000 C CNN
+F 1 "74HC393" H 7650 2126 50  0000 C CNN
 F 2 "Package_SO:TSSOP-14_4.4x5mm_P0.65mm" H 7650 1850 50  0001 C CNN
 F 3 "74xx\\74LS393.pdf" H 7650 1850 50  0001 C CNN
@@
 AR Path="/613AFF13/615372DE" Ref="U12"  Part="2"
 F 0 "U12" H 7650 3217 50  0000 C CNN
-F 1 "74LS393" H 7650 3126 50  0000 C CNN
+F 1 "74HC393" H 7650 3126 50  0000 C CNN
 F 2 "Package_SO:TSSOP-14_4.4x5mm_P0.65mm" H 7650 2850 50  0001 C CNN
 F 3 "74xx\\74LS393.pdf" H 7650 2850 50  0001 C CNN
@@
 AR Path="/613AFF13/61661DB1" Ref="U7"  Part="1"
 F 0 "U7" H 2700 7225 50  0000 C CNN
-F 1 "74LS32" H 2700 7134 50  0000 C CNN
+F 1 "74HC32" H 2700 7134 50  0000 C CNN
 F 2 "Package_SO:TSSOP-14_4.4x5mm_P0.65mm" H 2700 6900 50  0001 C CNN
 F 3 "http://www.ti.com/lit/gpn/sn74LS32" H 2700 6900 50  0001 C CNN
@@
 AR Path="/613AFF13/61C481DF" Ref="U7"  Part="2"
 F 0 "U7" H 3300 7475 50  0000 C CNN
-F 1 "74LS32" H 3300 7384 50  0000 C CNN
+F 1 "74HC32" H 3300 7384 50  0000 C CNN
 F 2 "Package_SO:TSSOP-14_4.4x5mm_P0.65mm" H 3300 7150 50  0001 C CNN
 F 3 "http://www.ti.com/lit/gpn/sn74LS32" H 3300 7150 50  0001 C CNN
@@
 P 5900 6700
 F 0 "U8" H 5900 7025 50  0000 C CNN
-F 1 "74LS08" H 5900 6934 50  0000 C CNN
+F 1 "74HC08" H 5900 6934 50  0000 C CNN
 F 2 "Package_SO:TSSOP-14_4.4x5mm_P0.65mm" H 5900 6700 50  0001 C CNN
 F 3 "http://www.ti.com/lit/gpn/sn74LS08" H 5900 6700 50  0001 C CNN
