File: hardware/k30-SBC/Memory.sch (KiCad schematic (older format))
At the start: 3 parts, among them U14 AS6C8016, U15 AS6C8016, U16 AM29F040

Commit message: Almost completed k30-SBC board design
Connections:
- net D0: no longer U15.13 (Q4), U15.29 (Q8), U15.35 (Q12)
- net D1: no longer U15.14 (Q5), U15.30 (Q9), U15.36 (Q13)
- net D2: no longer U15.15 (Q6), U15.31 (Q10), U15.37 (Q14)
- net D3: no longer U15.16 (Q7), U15.32 (Q11), U15.38 (Q15)
- new net D10: U15.31 (Q10)
- new net D11: U15.32 (Q11)
- new net D12: U15.35 (Q12)
- new net D13: U15.36 (Q13)
- new net D14: U15.37 (Q14)
- new net D15: U15.38 (Q15)
- new net D4: U15.13 (Q4)
- new net D5: U15.14 (Q5)
- new net D6: U15.15 (Q6)
- new net D7: U15.16 (Q7)
- new net D8: U15.29 (Q8)
- new net D9: U15.30 (Q9)
Changed lines of the file:
@@
 	3500 4950 3750 4950
 Text Label 3750 4950 2    50   ~ 0
-D0
+D4
 Entry Wire Line
 	3750 5050 3850 4950
@@
 	3500 5050 3750 5050
 Text Label 3750 5050 2    50   ~ 0
-D1
+D5
 Entry Wire Line
 	3750 5150 3850 5050
@@
 	3500 5150 3750 5150
 Text Label 3750 5150 2    50   ~ 0
-D2
+D6
 Entry Wire Line
 	3750 5250 3850 5150
@@
 	3500 5250 3750 5250
 Text Label 3750 5250 2    50   ~ 0
-D3
+D7
 Entry Wire Line
 	3750 5350 3850 5250
@@
 	3500 5350 3750 5350
 Text Label 3750 5350 2    50   ~ 0
-D0
+D8
 Entry Wire Line
 	3750 5450 3850 5350
@@
 	3500 5450 3750 5450
 Text Label 3750 5450 2    50   ~ 0
-D1
+D9
 Entry Wire Line
 	3750 5550 3850 5450
@@
 	3500 5550 3750 5550
 Text Label 3750 5550 2    50   ~ 0
-D2
+D10
 Entry Wire Line
 	3750 5650 3850 5550
@@
 	3500 5650 3750 5650
 Text Label 3750 5650 2    50   ~ 0
-D3
+D11
 Entry Wire Line
 	3750 5750 3850 5650
@@
 	3500 5750 3750 5750
 Text Label 3750 5750 2    50   ~ 0
-D0
+D12
 Entry Wire Line
 	3750 5850 3850 5750
@@
 	3500 5850 3750 5850
 Text Label 3750 5850 2    50   ~ 0
-D1
+D13
 Entry Wire Line
 	3750 5950 3850 5850
@@
 	3500 5950 3750 5950
 Text Label 3750 5950 2    50   ~ 0
-D2
+D14
 Entry Wire Line
 	3750 6050 3850 5950
@@
 	3500 6050 3750 6050
 Text Label 3750 6050 2    50   ~ 0
-D3
+D15
 $Comp
 L ComputieParts:AM29F040 U16
