File: hardware/k30-SBC/IO.sch (KiCad schematic (older format))
At the start: 26 parts, among them J1 CompactFlash, J2 Serial1, J3 Serial2, SW3 IP2, SW4 IP3, U13 MC68681, U7 74LS32, Y2 Crystal

Commit message: Almost completed k30-SBC board design
Parts:
- U7: value 74LS32 -> 74HC32
Connections:
- net A0 is gone; now on net A1: U13.2 (RS1)
- net D0 is gone; now on net D24: J1.21 (Pin_21)
- net D1 is gone; now on net D25: J1.22 (Pin_22)
- net D2 is gone; now on net D26: J1.23 (Pin_23)
- net D3 is gone; now on net D27: J1.2 (Pin_2)
- net D4 is gone; now on net D28: J1.3 (Pin_3)
- net D5 is gone; now on net D29: J1.4 (Pin_4)
- net D6 is gone; now on net D30: J1.5 (Pin_5)
- net D7 is gone; now on net D31: J1.6 (Pin_6)
- net A1: no longer U13.4 (RS2)
- net A2: now also U13.4 (RS2); no longer U13.6 (RS3)
- net A3: now also U13.6 (RS3); no longer U13.7 (RS4)
- net A4: now also U13.7 (RS4)
- net D10: no longer names the net of J1.49 (Pin_49)
- net D11: no longer names the net of J1.27 (Pin_27)
- net D12: no longer names the net of J1.28 (Pin_28)
- net D13: no longer names the net of J1.29 (Pin_29)
- net D14: no longer names the net of J1.30 (Pin_30)
- net D15: no longer names the net of J1.31 (Pin_31)
- net D8: no longer names the net of J1.47 (Pin_47)
- net D9: no longer names the net of J1.48 (Pin_48)
Changed lines of the file:
@@
 	3050 2750 2950 2650
 Text Label 3050 2450 0    50   ~ 0
-A0
+A1
 Text Label 3050 2550 0    50   ~ 0
-A1
+A2
 Text Label 3050 2650 0    50   ~ 0
-A2
+A3
 Text Label 3050 2750 0    50   ~ 0
-A3
+A4
 Wire Wire Line
 	4000 2450 3050 2450
@@
 	4200 5450 4100 5350
 Text Label 4200 5050 0    50   ~ 0
-D3
+D27
 Text Label 4200 5150 0    50   ~ 0
-D4
+D28
 Text Label 4200 5250 0    50   ~ 0
-D5
+D29
 Text Label 4200 5350 0    50   ~ 0
-D6
+D30
 Text Label 4200 5450 0    50   ~ 0
-D7
+D31
 Wire Wire Line
 	4750 5050 4200 5050
@@
 	4200 7150 4100 7050
 Text Label 4200 6950 0    50   ~ 0
-D0
+D24
 Text Label 4200 7050 0    50   ~ 0
-D1
+D25
 Text Label 4200 7150 0    50   ~ 0
-D2
+D26
 Wire Wire Line
 	4750 6950 4200 6950
@@
 Wire Wire Line
 	4750 7150 4200 7150
-Entry Wire Line
-	5800 5050 5900 4950
-Entry Wire Line
-	5800 5150 5900 5050
-Entry Wire Line
-	5800 7050 5900 6950
-Entry Wire Line
-	5800 7150 5900 7050
-Entry Wire Line
-	5800 7250 5900 7150
-Text Label 5800 5050 2    50   ~ 0
-D11
-Text Label 5800 5150 2    50   ~ 0
-D12
-Text Label 5800 7050 2    50   ~ 0
-D8
-Text Label 5800 7150 2    50   ~ 0
-D9
-Text Label 5800 7250 2    50   ~ 0
-D10
-Wire Wire Line
-	5250 5050 5800 5050
-Wire Wire Line
-	5250 5150 5800 5150
-Wire Wire Line
-	5250 7050 5800 7050
-Wire Wire Line
-	5250 7150 5800 7150
-Wire Wire Line
-	5250 7250 5800 7250
-Entry Wire Line
-	5800 5250 5900 5150
-Entry Wire Line
-	5800 5350 5900 5250
-Text Label 5800 5250 2    50   ~ 0
-D13
-Text Label 5800 5350 2    50   ~ 0
-D14
-Wire Wire Line
-	5250 5250 5800 5250
-Wire Wire Line
-	5250 5350 5800 5350
-Entry Wire Line
-	5800 5450 5900 5350
-Text Label 5800 5450 2    50   ~ 0
-D15
-Wire Wire Line
-	5250 5450 5800 5450
-Wire Bus Line
-	4100 4400 5900 4400
-Connection ~ 4100 4400
 Wire Wire Line
 	4550 6150 4750 6150
@@
 AR Path="/613CC863/625F92BB" Ref="U7"  Part="3"
 F 0 "U7" H 2500 5825 50  0000 C CNN
-F 1 "74LS32" H 2500 5734 50  0000 C CNN
+F 1 "74HC32" H 2500 5734 50  0000 C CNN
 F 2 "Package_SO:TSSOP-14_4.4x5mm_P0.65mm" H 2500 5500 50  0001 C CNN
 F 3 "http://www.ti.com/lit/gpn/sn74LS32" H 2500 5500 50  0001 C CNN
@@
 AR Path="/613CC863/62603C2A" Ref="U7"  Part="4"
 F 0 "U7" H 2500 6375 50  0000 C CNN
-F 1 "74LS32" H 2500 6284 50  0000 C CNN
+F 1 "74HC32" H 2500 6284 50  0000 C CNN
 F 2 "Package_SO:TSSOP-14_4.4x5mm_P0.65mm" H 2500 6050 50  0001 C CNN
 F 3 "http://www.ti.com/lit/gpn/sn74LS32" H 2500 6050 50  0001 C CNN
@@
 	2950 1100 2950 2650
 Wire Bus Line
-	5900 4400 5900 7150
-Wire Bus Line
 	4100 4400 4100 7050

Commit message: Fixed CF footprint and the wrong data pins going for CF
Parts:
- J2, J3: footprint Connector_PinHeader_2.54mm:PinHeader_1x06_P2.54mm_Horizontal -> Connector_PinHeader_2.54mm:PinHeader_1x06_P2.54mm_Vertical
Changed lines of the file:
@@
 F 0 "J2" H 9022 1224 50  0000 R CNN
 F 1 "Serial1" H 9022 1133 50  0000 R CNN
-F 2 "Connector_PinHeader_2.54mm:PinHeader_1x06_P2.54mm_Horizontal" H 9050 1250 50  0001 C CNN
+F 2 "Connector_PinHeader_2.54mm:PinHeader_1x06_P2.54mm_Vertical" H 9050 1250 50  0001 C CNN
 F 3 "~" H 9050 1250 50  0001 C CNN
 	1    9050 1250
@@
 F 0 "J3" H 9078 2326 50  0000 L CNN
 F 1 "Serial2" H 9078 2235 50  0000 L CNN
-F 2 "Connector_PinHeader_2.54mm:PinHeader_1x06_P2.54mm_Horizontal" H 9050 2350 50  0001 C CNN
+F 2 "Connector_PinHeader_2.54mm:PinHeader_1x06_P2.54mm_Vertical" H 9050 2350 50  0001 C CNN
 F 3 "~" H 9050 2350 50  0001 C CNN
 	1    9050 2350
