File: hardware/k30-SBC/Bus.kicad_sch (KiCad schematic)
At the start: 31 parts, among them J4 ADBUS-EXP, J5 ADBUS, J6 SIGBUS, J7 POWER, J8 POWER, J9 POWER, U12 74HC393, U2 74HC14, U3 74HC05, U4 74HC139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

Commit message: Revision 2 of k30-SBC
Connections:
- net 0SEL renamed ~{0SEL}
- net 3SEL renamed ~{3SEL}
- net 4SEL renamed ~{4SEL}
- net 5SEL renamed ~{5SEL}
- net 6SEL renamed ~{6SEL}
- net AS renamed ~{AS}
- net AVEC renamed ~{AVEC}
- net BERR renamed ~{BERR}
- net BG renamed ~{BG}
- net BGACK renamed ~{BGACK}
- net BR renamed ~{BR}
- net DS renamed ~{DS}
- net DSACK0 renamed ~{DSACK0}
- net DSACK1 renamed ~{DSACK1}
- net HALT renamed ~{HALT}
- net IACK renamed ~{IACK}
- net IOSEL renamed ~{IOSEL}
- net IPL0 renamed ~{IPL0}
- net IPL1 renamed ~{IPL1}
- net IPL2 renamed ~{IPL2}
- net RAMSEL renamed ~{RAMSEL}
- net RD renamed ~{RD}
- net RESET renamed ~{RESET}
- net ROMSEL renamed ~{ROMSEL}
- net WR renamed ~{WR}
