File: hardware/k30-SBC/IO.kicad_sch (KiCad schematic)
At the start: 26 parts, among them J1 CompactFlash, J2 Serial1, J3 Serial2, SW3 IP2, SW4 IP3, U13 MC68681, U7 74HC32, Y2 Crystal

Commit message: Upgraded project formats to kicad 6.0
Parts:
- J1: footprint 68k-SMT:CF-Card_3M_N7E50-Q516RB-40 -> Computie_Connectors:CF-Card_3M_N7E50-Q516RB-40
- U13: footprint Package_LCC:PLCC-44_THT-Socket -> Package_LCC:PLCC-68_THT-Socket; symbol ComputieParts:68681-PLCC -> Computie_68k:MC68681-PLCC
Changed lines of the file:
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@@
     (pin "2")
   )
-  (symbol (lib_id "ComputieParts:68681-PLCC") (at 127 62.23 0) (unit 1)
+  (symbol (lib_id "Computie_68k:MC68681-PLCC") (at 127 62.23 0) (unit 1)
     (in_bom yes) (on_board yes)
     (property "Reference" "U13" (id 0) (at 127 19.5326 0))
     (property "Value" "MC68681" (id 1) (at 127 21.844 0))
-    (property "Footprint" "Package_LCC:PLCC-44_THT-Socket" (id 2) (at 127 62.23 0)
+    (property "Footprint" "Package_LCC:PLCC-68_THT-Socket" (id 2) (at 127 62.23 0)
       (effects (font (size 1.27 1.27)) hide)
     )
@@
     (property "Reference" "J1" (id 0) (at 127 120.2182 0))
     (property "Value" "CompactFlash" (id 1) (at 127 122.5296 0))
-    (property "Footprint" "68k-SMT:CF-Card_3M_N7E50-Q516RB-40" (id 2) (at 125.73 156.21 0)
+    (property "Footprint" "Computie_Connectors:CF-Card_3M_N7E50-Q516RB-40" (id 2) (at 125.73 156.21 0)
       (effects (font (size 1.27 1.27)) hide)
     )

Commit message: Revision 2 of k30-SBC
Parts:
- JP3: value IACK -> ~{IACK}
- U13: footprint Package_LCC:PLCC-68_THT-Socket -> Package_LCC:PLCC-44_THT-Socket
Connections:
- net 6SEL renamed ~{6SEL}
- net DSACK0 renamed ~{DSACK0}
- net IACK renamed ~{IACK}
- net IORD renamed ~{IORD}
- net IOSEL renamed ~{IOSEL}
- net IOWR renamed ~{IOWR}
- net IPL1 renamed ~{IPL1}
- net RD renamed ~{RD}
- net RESET renamed ~{RESET}
- net SIACK renamed ~{SIACK}
- net SIRQ renamed ~{SIRQ}
- net WR renamed ~{WR}
Changed lines of the file:
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@@
   (title_block
     (title "k30 SBC")
-    (rev "1")
+    (rev "2")
   )
   (junction (at 119.38 158.75) (diameter 0) (color 0 0 0 0)
@@
     (effects (font (size 1.27 1.27)) (justify left bottom))
   )
-  (global_label "WR" (shape input) (at 95.25 77.47 180) (fields_autoplaced)
+  (global_label "~{WR}" (shape input) (at 95.25 77.47 180) (fields_autoplaced)
     (effects (font (size 1.27 1.27)) (justify right))
     (property "Intersheet References" "${INTERSHEET_REFS}" (id 0) (at 0 0 0)
@@
     )
   )
-  (global_label "IORD" (shape input) (at 138.43 146.05 0) (fields_autoplaced)
+  (global_label "~{IORD}" (shape input) (at 138.43 146.05 0) (fields_autoplaced)
     (effects (font (size 1.27 1.27)) (justify left))
     (property "Intersheet References" "${INTERSHEET_REFS}" (id 0) (at 0 0 0)
@@
     )
   )
-  (global_label "IOSEL" (shape input) (at 95.25 74.93 180) (fields_autoplaced)
-    (effects (font (size 1.27 1.27)) (justify right))
-    (property "Intersheet References" "${INTERSHEET_REFS}" (id 0) (at 0 0 0)
-      (effects (font (size 1.27 1.27)) hide)
-    )
-  )
-  (global_label "IORD" (shape input) (at 76.2 139.7 0) (fields_autoplaced)
+  (global_label "~{IOSEL}" (shape input) (at 95.25 74.93 180) (fields_autoplaced)
+    (effects (font (size 1.27 1.27)) (justify right))
+    (property "Intersheet References" "${INTERSHEET_REFS}" (id 0) (at 0 0 0)
+      (effects (font (size 1.27 1.27)) hide)
+    )
+  )
+  (global_label "~{IORD}" (shape input) (at 76.2 139.7 0) (fields_autoplaced)
     (effects (font (size 1.27 1.27)) (justify left))
     (property "Intersheet References" "${INTERSHEET_REFS}" (id 0) (at 0 0 0)
@@
     )
   )
-  (global_label "6SEL" (shape input) (at 49.53 137.16 180) (fields_autoplaced)
-    (effects (font (size 1.27 1.27)) (justify right))
-    (property "Intersheet References" "${INTERSHEET_REFS}" (id 0) (at 0 0 0)
-      (effects (font (size 1.27 1.27)) hide)
-    )
-  )
-  (global_label "6SEL" (shape input) (at 49.53 151.13 180) (fields_autoplaced)
-    (effects (font (size 1.27 1.27)) (justify right))
-    (property "Intersheet References" "${INTERSHEET_REFS}" (id 0) (at 0 0 0)
-      (effects (font (size 1.27 1.27)) hide)
-    )
-  )
-  (global_label "SIACK" (shape input) (at 95.25 80.01 180) (fields_autoplaced)
-    (effects (font (size 1.27 1.27)) (justify right))
-    (property "Intersheet References" "${INTERSHEET_REFS}" (id 0) (at 0 0 0)
-      (effects (font (size 1.27 1.27)) hide)
-    )
-  )
-  (global_label "SIRQ" (shape input) (at 67.31 80.01 0) (fields_autoplaced)
+  (global_label "~{6SEL}" (shape input) (at 49.53 137.16 180) (fields_autoplaced)
+    (effects (font (size 1.27 1.27)) (justify right))
+    (property "Intersheet References" "${INTERSHEET_REFS}" (id 0) (at 0 0 0)
+      (effects (font (size 1.27 1.27)) hide)
+    )
+  )
+  (global_label "~{6SEL}" (shape input) (at 49.53 151.13 180) (fields_autoplaced)
+    (effects (font (size 1.27 1.27)) (justify right))
+    (property "Intersheet References" "${INTERSHEET_REFS}" (id 0) (at 0 0 0)
+      (effects (font (size 1.27 1.27)) hide)
+    )
+  )
+  (global_label "~{SIACK}" (shape input) (at 95.25 80.01 180) (fields_autoplaced)
+    (effects (font (size 1.27 1.27)) (justify right))
+    (property "Intersheet References" "${INTERSHEET_REFS}" (id 0) (at 0 0 0)
+      (effects (font (size 1.27 1.27)) hide)
+    )
+  )
+  (global_label "~{SIRQ}" (shape input) (at 67.31 80.01 0) (fields_autoplaced)
     (effects (font (size 1.27 1.27)) (justify left))
     (property "Intersheet References" "${INTERSHEET_REFS}" (id 0) (at -2.54 0 0)
@@
     )
   )
-  (global_label "SIRQ" (shape output) (at 95.25 90.17 180) (fields_autoplaced)
-    (effects (font (size 1.27 1.27)) (justify right))
-    (property "Intersheet References" "${INTERSHEET_REFS}" (id 0) (at 0 0 0)
-      (effects (font (size 1.27 1.27)) hide)
-    )
-  )
-  (global_label "IACK" (shape input) (at 49.53 90.17 180) (fields_autoplaced)
+  (global_label "~{SIRQ}" (shape output) (at 95.25 90.17 180) (fields_autoplaced)
+    (effects (font (size 1.27 1.27)) (justify right))
+    (property "Intersheet References" "${INTERSHEET_REFS}" (id 0) (at 0 0 0)
+      (effects (font (size 1.27 1.27)) hide)
+    )
+  )
+  (global_label "~{IACK}" (shape input) (at 49.53 90.17 180) (fields_autoplaced)
     (effects (font (size 1.27 1.27)) (justify right))
     (property "Intersheet References" "${INTERSHEET_REFS}" (id 0) (at 2.54 0 0)
@@
     )
   )
-  (global_label "IOWR" (shape input) (at 76.2 153.67 0) (fields_autoplaced)
+  (global_label "~{IOWR}" (shape input) (at 76.2 153.67 0) (fields_autoplaced)
     (effects (font (size 1.27 1.27)) (justify left))
     (property "Intersheet References" "${INTERSHEET_REFS}" (id 0) (at 0 0 0)
@@
     )
   )
-  (global_label "DSACK0" (shape input) (at 95.25 87.63 180) (fields_autoplaced)
-    (effects (font (size 1.27 1.27)) (justify right))
-    (property "Intersheet References" "${INTERSHEET_REFS}" (id 0) (at 0 0 0)
-      (effects (font (size 1.27 1.27)) hide)
-    )
-  )
-  (global_label "RD" (shape input) (at 49.53 142.24 180) (fields_autoplaced)
+  (global_label "~{DSACK0}" (shape input) (at 95.25 87.63 180) (fields_autoplaced)
+    (effects (font (size 1.27 1.27)) (justify right))
+    (property "Intersheet References" "${INTERSHEET_REFS}" (id 0) (at 0 0 0)
+      (effects (font (size 1.27 1.27)) hide)
+    )
+  )
+  (global_label "~{RD}" (shape input) (at 49.53 142.24 180) (fields_autoplaced)
     (effects (font (size 1.27 1.27)) (justify right))
     (property "Intersheet References" "${INTERSHEET_REFS}" (id 0) (at 0 0 0)
@@
     )
   )
-  (global_label "RESET" (shape input) (at 138.43 163.83 0) (fields_autoplaced)
+  (global_label "~{RESET}" (shape input) (at 138.43 163.83 0) (fields_autoplaced)
     (effects (font (size 1.27 1.27)) (justify left))
     (property "Intersheet References" "${INTERSHEET_REFS}" (id 0) (at 146.4994 163.7506 0)
@@
     )
   )
-  (global_label "IOWR" (shape input) (at 138.43 148.59 0) (fields_autoplaced)
+  (global_label "~{IOWR}" (shape input) (at 138.43 148.59 0) (fields_autoplaced)
     (effects (font (size 1.27 1.27)) (justify left))
     (property "Intersheet References" "${INTERSHEET_REFS}" (id 0) (at 0 0 0)
@@
     )
   )
-  (global_label "IPL1" (shape output) (at 49.53 80.01 180) (fields_autoplaced)
+  (global_label "~{IPL1}" (shape output) (at 49.53 80.01 180) (fields_autoplaced)
     (effects (font (size 1.27 1.27)) (justify right))
     (property "Intersheet References" "${INTERSHEET_REFS}" (id 0) (at 2.54 0 0)
@@
     )
   )
-  (global_label "SIACK" (shape output) (at 67.31 90.17 0) (fields_autoplaced)
+  (global_label "~{SIACK}" (shape output) (at 67.31 90.17 0) (fields_autoplaced)
     (effects (font (size 1.27 1.27)) (justify left))
     (property "Intersheet References" "${INTERSHEET_REFS}" (id 0) (at -2.54 0 0)
@@
     )
   )
-  (global_label "WR" (shape input) (at 49.53 156.21 180) (fields_autoplaced)
-    (effects (font (size 1.27 1.27)) (justify right))
-    (property "Intersheet References" "${INTERSHEET_REFS}" (id 0) (at 0 0 0)
-      (effects (font (size 1.27 1.27)) hide)
-    )
-  )
-  (global_label "RESET" (shape input) (at 95.25 82.55 180) (fields_autoplaced)
+  (global_label "~{WR}" (shape input) (at 49.53 156.21 180) (fields_autoplaced)
+    (effects (font (size 1.27 1.27)) (justify right))
+    (property "Intersheet References" "${INTERSHEET_REFS}" (id 0) (at 0 0 0)
+      (effects (font (size 1.27 1.27)) hide)
+    )
+  )
+  (global_label "~{RESET}" (shape input) (at 95.25 82.55 180) (fields_autoplaced)
     (effects (font (size 1.27 1.27)) (justify right))
     (property "Intersheet References" "${INTERSHEET_REFS}" (id 0) (at 0 0 0)
@@
     (property "Reference" "U13" (id 0) (at 127 19.5326 0))
     (property "Value" "MC68681" (id 1) (at 127 21.844 0))
-    (property "Footprint" "Package_LCC:PLCC-68_THT-Socket" (id 2) (at 127 62.23 0)
+    (property "Footprint" "Package_LCC:PLCC-44_THT-Socket" (id 2) (at 127 62.23 0)
       (effects (font (size 1.27 1.27)) hide)
     )
@@
     (in_bom yes) (on_board yes)
     (property "Reference" "JP3" (id 0) (at 58.42 83.4644 0))
-    (property "Value" "IACK" (id 1) (at 58.42 85.7758 0))
+    (property "Value" "~{IACK}" (id 1) (at 58.42 85.7758 0))
     (property "Footprint" "Connector_PinHeader_2.54mm:PinHeader_1x02_P2.54mm_Vertical" (id 2) (at 58.42 90.17 0)
       (effects (font (size 1.27 1.27)) hide)
