File: hardware/k30-SBC/Logic.kicad_sch (KiCad schematic)
At the start: 20 parts, among them SW2 SW_DIP_x06, U10 74HC253, U11 74HC138, U12 74HC393, U17 74LVC1G32, U2 74HC14, U3 74HC05, U4 74HC139, U5 4072, U6 74HC20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

Commit message: Revision 2 of k30-SBC
Parts:
- TP4: value DSACK-EXT -> ~{DSACK-EXT}
- TP8: value DSACK-SEL -> ~{DSACK-SEL}
- gave numbers to parts that had none: 1
Connections:
- net 0SEL renamed ~{0SEL}
- net 3SEL renamed ~{3SEL}
- net 4SEL renamed ~{4SEL}
- net 5SEL renamed ~{5SEL}
- net 6SEL renamed ~{6SEL}
- net AS renamed ~{AS}
- net ATA-DSACK renamed ~{ATA-DSACK}
- net BERR renamed ~{BERR}
- net CDIS renamed ~{CDIS}
- net DS renamed ~{DS}
- net DSACK-EXT renamed ~{DSACK-EXT}
- net DSACK0 renamed ~{DSACK0}
- net DSACK1 renamed ~{DSACK1}
- net IACK renamed ~{IACK}
- net IOSEL renamed ~{IOSEL}
- net MMUDIS renamed ~{MMUDIS}
- net RAMSEL renamed ~{RAMSEL}
- net ROMSEL renamed ~{ROMSEL}
