File: hardware/k30-SBC/k30-SBC.kicad_sch (KiCad schematic)
At the start: 18 parts, among them SW1 RESET, U1 MC68030FE, U2 74HC14, U3 74HC05, Y1 Crystal

Commit message: Upgraded project formats to kicad 6.0
Parts:
- U1: symbol ComputieParts:MC68030FE -> Computie_68k:MC68030FE
Changed lines of the file:
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@@
     )
   )
-  (symbol (lib_id "ComputieParts:MC68030FE") (at 93.98 104.14 0) (unit 1)
+  (symbol (lib_id "Computie_68k:MC68030FE") (at 93.98 104.14 0) (unit 1)
     (in_bom yes) (on_board yes)
     (property "Reference" "U1" (id 0) (at 67.31 19.05 0))
@@
     )
     (path "/00000000-0000-0000-0000-0000613cc863/00000000-0000-0000-0000-0000614fafb4"
-      (reference "J1") (unit 1) (value "CompactFlash") (footprint "68k-SMT:CF-Card_3M_N7E50-Q516RB-40")
+      (reference "J1") (unit 1) (value "CompactFlash") (footprint "Computie_Connectors:CF-Card_3M_N7E50-Q516RB-40")
     )
     (path "/00000000-0000-0000-0000-0000613cc863/00000000-0000-0000-0000-0000613d9ce3"
@@
     )
     (path "/00000000-0000-0000-0000-0000613cc863/00000000-0000-0000-0000-0000613d9dae"
-      (reference "U13") (unit 1) (value "MC68681") (footprint "Package_LCC:PLCC-44_THT-Socket")
+      (reference "U13") (unit 1) (value "MC68681") (footprint "Package_LCC:PLCC-68_THT-Socket")
     )
     (path "/00000000-0000-0000-0000-0000613dffc0/00000000-0000-0000-0000-0000613f02a2"

Commit message: Revision 2 of k30-SBC
Parts:
- SW1: value RESET -> ~{RESET}
Connections:
- net AS renamed ~{AS}
- net AVEC renamed ~{AVEC}
- net BERR renamed ~{BERR}
- net BG renamed ~{BG}
- net BGACK renamed ~{BGACK}
- net BR renamed ~{BR}
- net CDIS renamed ~{CDIS}
- net DS renamed ~{DS}
- net DSACK-EXT renamed ~{DSACK-EXT}
- net DSACK0 renamed ~{DSACK0}
- net DSACK1 renamed ~{DSACK1}
- net HALT renamed ~{HALT}
- net IPL0 renamed ~{IPL0}
- net IPL1 renamed ~{IPL1}
- net IPL2 renamed ~{IPL2}
- net MMUDIS renamed ~{MMUDIS}
- net RD renamed ~{RD}
- net RESET renamed ~{RESET}
- net WR renamed ~{WR}
