File: hardware/68k-Supervisor/68kBoardSupervisorShield.kicad_pcb (KiCad board)
At the start: 2 copper layers, 89.9 x 53.3 mm, 6 parts, among them J1 ADBUS, J2 SIGBUS, J3 UNMAPPED, SW1 RESET

Commit message: Upgraded project formats to kicad 6.0
Connections:
- net R~W renamed R~{W}
Other:
- net class Default removed
- board text added: "R/~{W }"
- board text added: "R/~{W}"
- board text removed: "R/~W"
